Commit message: Update phantomX_model.xacro

File: hexapod_description/urdf/phantomX_model.xacro (robot description, xacro)
@@ -51,5 +51,5 @@
     </gazebo>
 	<!-- Head Pan and Tilt properties -->
-	<joint name="head_pan_joint" type="revolute">
+	<joint name="head_pan_joint" type="fixed">
 		<parent link="body_link"/>
 		<child link="head_pan_link"/>
@@ -68,5 +68,5 @@
         </inertial>
     </link>
-	<joint name="head_tilt_joint" type="revolute">
+	<joint name="head_tilt_joint" type="fixed">
 		<parent link="head_pan_link"/>
 		<child link="head_tilt_link"/>

Commit message: Update phantomX_model.xacro
Adapted the IMU Position in imu_link

File: hexapod_description/urdf/phantomX_model.xacro (robot description, xacro)
@@ -137,14 +137,5 @@
 		<origin xyz="0.0 0.0 0.0" rpy="0.0 0.0 0.0" />
 	</joint>
-	<link name="imu_link">
-        <inertial>
-            <origin xyz="0.0 0.0 0.0" rpy="0.0 0.0 0.0" />
-            <mass value="0.00001"/>
-            <inertia
-                ixx="1.0" ixy="0.0"  ixz="0.0"
-                iyy="1.0" iyz="0.0"
-                izz="1.0" />
-        </inertial>
-    </link>
+	<link name="imu_link" />
 	<!-- Joint properties -->
 	<xacro:property name="joint_lower_limit" value="-${3.14}" />

Commit message: Update phantomX_model.xacro

File: hexapod_description/urdf/phantomX_model.xacro (robot description, xacro)
@@ -131,4 +131,18 @@
         </inertial>
     </link>
+<!-- Laser properties -->
+ <joint name="base_to_laser" type="fixed">
+      <parent link="base_link"/>
+      <child link="laser"/>
+      <origin xyz="0.065 0.0 0.1960"/>
+ </joint>
+ <link name="laser">
+       <visual>
+        <geometry>
+          <cylinder length="0.04" radius="0.04"/>
+        </geometry>
+        <material name="black"/>
+      </visual>
+ </link>
 	<!-- IMU properties -->
 	<joint name="imu_joint" type="fixed">

Commit message: Add files via upload

File: hexapod_description/urdf/phantomX_model.xacro (robot description, xacro)
@@ -135,5 +135,5 @@
       <parent link="base_link"/>
       <child link="laser"/>
-      <origin xyz="0.065 0.0 0.1960"/>
+      <origin xyz="0.0 0.0 0.1960"/>
  </joint>
  <link name="laser">
@@ -151,5 +151,14 @@
 		<origin xyz="0.0 0.0 0.0" rpy="0.0 0.0 0.0" />
 	</joint>
-	<link name="imu_link" />
+	<link name="imu_link">
+<!--        <inertial>
+            <origin xyz="0.0 0.0 0.0" rpy="0.0 0.0 0.0" />
+            <mass value="0.00001"/>
+            <inertia
+                ixx="1.0" ixy="0.0"  ixz="0.0"
+                iyy="1.0" iyz="0.0"
+                izz="1.0" />
+        </inertial> -->
+    </link>
 	<!-- Joint properties -->
 	<xacro:property name="joint_lower_limit" value="-${3.14}" />
